File: rutten_motor_board.brd (EAGLE design)
At the start: 68.6 x 53.3 mm, 14 parts, among them U1 A4988_STEP_STICK, U2 A4988_STEP_STICK, U3 XBee Connector

Commit message: Finalized layout
Parts:
- added JP6: 5V OUT, screwterms:SCREW_TERM-200MIL-2
- JP1, JP2, JP3, JP4, JP5: device microbuilder:TERMBLOCK_1X2-3.5MM -> screwterms:SCREW_TERM-200MIL-2
- moved JP2 9.98 mm to (13.2, 31.0)
- moved JP1 8.03 mm to (13.2, 41.1)
- moved C1 3.97 mm to (14.2, 19.3), turned to 90 degrees
- moved JP4 3.30 mm to (58.2, 43.2)
- moved JP3 1.27 mm to (58.2, 33.0)
- moved JP5 1.27 mm to (4.57, 18.0)
- moved U3 0.57 mm to (65.3, 17.8), turned to 270 degrees
Connections:
- removed net 1-RES: U1.RES
- removed net 2-RES: U2.RES
- net +12V: now also JP5.P$2; no longer JP5.1
- net +5V: now also JP6.P$2, U1.RES, U2.RES
- net 1-A1: now also JP1.P$2; no longer JP1.1
- net 1-A2: now also JP1.P$1; no longer JP1.2
- net 1-B1: now also JP2.P$2; no longer JP2.1
- net 1-B2: now also JP2.P$1; no longer JP2.2
- net 2-A1: now also JP3.P$2; no longer JP3.1
- net 2-A2: now also JP3.P$1; no longer JP3.2
- net 2-B1: now also JP4.P$2; no longer JP4.1
- net 2-B2: now also JP4.P$1; no longer JP4.2
- net GND: now also JP5.P$1, JP6.P$1; no longer JP5.2
Routing:
- net XB-TX: track 28.9 -> 43.8 mm, vias 0 -> 1
- net +12V: track 79.4 -> 67.1 mm
- net 1-B2: track 25.7 -> 37.1 mm, vias 2 -> 3
- net XB-RX: track 32.5 -> 41.9 mm, vias 0 -> 2
- net 1-A1: track 36.3 -> 28.5 mm, vias 3 -> 0
- net GND: track 6.85 -> 0.00 mm
- net 2-B2: track 39.9 -> 46.0 mm, vias 1 -> 3
- net 1-B1: track 26.7 -> 32.5 mm
- net 2-A1: track 31.2 -> 25.7 mm, vias 3 -> 2
- net 2-A2: track 25.2 -> 28.2 mm
- net 2-B1: track 49.5 -> 47.0 mm
- net 2-MS3: track 48.6 -> 50.4 mm
- net 2-DIR: track 76.6 -> 75.1 mm
- net 1-A2: track 35.3 -> 34.5 mm
- net 1-MS3: track 32.7 -> 33.0 mm, vias 0 -> 1
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Other:
- board text added: "+12V IN"
- board text added: "+5V OUT"
- board text added: "1-A"
- board text added: "1-A'"
- board text added: "1-B"
- board text added: "1-B'"
- board text added: "2-A"
- board text added: "2-A'"
- board text added: "2-B"
- board text added: "2-B'"
- board text added: "C1"
- board text added: "GND"
