File: rutten_motor_board.sch (EAGLE design)
At the start: 14 parts, among them U1 A4988_STEP_STICK, U2 A4988_STEP_STICK, U3 XBee Connector

Commit message: Finalized layout
Parts:
- added JP6: 5V OUT, screwterms:SCREWTERM-2
- JP1, JP2, JP3, JP4, JP5: device microbuilder:TERMBLOCK_1X2 -> screwterms:SCREWTERM-2
Connections:
- removed net 1-RES: U1.RES
- removed net 2-RES: U2.RES
- net +12V: now also JP5.2; no longer JP5.1
- net +5V: now also JP6.2, U1.RES, U2.RES
- net 1-A1: now also JP1.2; no longer JP1.1
- net 1-A2: now also JP1.1; no longer JP1.2
- net 1-B1: now also JP2.2; no longer JP2.1
- net 1-B2: now also JP2.1; no longer JP2.2
- net 2-A1: now also JP3.2; no longer JP3.1
- net 2-A2: now also JP3.1; no longer JP3.2
- net 2-B1: now also JP4.2; no longer JP4.1
- net 2-B2: now also JP4.1; no longer JP4.2
- net GND: now also JP5.1, JP6.1; no longer JP5.2
Other:
- note removed: "0.9V REF = -180°C to 820°C"
- note removed: "0V REF = 0°C to 1000°C"
- note removed: "1.24V REF = -248°C to 752°C"
- note removed: "J-Type Range = -180°C to 750°C"
- note removed: "K-Type Range = -180°C to 1200°C"
- note removed: "With a Single 5V Supply:"
Changed lines of the file:
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@@
 <part name="U$8" library="GeekAmmo" deviceset="FRAME2-A4" device=""/>
 <part name="U$9" library="GeekAmmo" deviceset="DOCFIELD1" device=""/>
-<part name="JP1" library="microbuilder" deviceset="TERMBLOCK_1X2" device="" value="Motor 1-A"/>
+<part name="JP1" library="screwterms" deviceset="SCREWTERM-2" device="" value="Motor 1-A"/>
 <part name="U1" library="Custom" deviceset="A4988_STEP_STICK" device=""/>
 <part name="U2" library="Custom" deviceset="A4988_STEP_STICK" device=""/>
-<part name="JP2" library="microbuilder" deviceset="TERMBLOCK_1X2" device="" value="Motor 1-B"/>
-<part name="JP3" library="microbuilder" deviceset="TERMBLOCK_1X2" device="" value="Motor 2-A"/>
-<part name="JP4" library="microbuilder" deviceset="TERMBLOCK_1X2" device="" value="Motor 2-B"/>
-<part name="JP5" library="microbuilder" deviceset="TERMBLOCK_1X2" device="" value="Motor Power"/>
+<part name="JP2" library="screwterms" deviceset="SCREWTERM-2" device="" value="Motor 1-B"/>
+<part name="JP3" library="screwterms" deviceset="SCREWTERM-2" device="" value="Motor 2-A"/>
+<part name="JP4" library="screwterms" deviceset="SCREWTERM-2" device="" value="Motor 2-B"/>
+<part name="JP5" library="screwterms" deviceset="SCREWTERM-2" device="" value="Motor Power"/>
 <part name="C1" library="SparkFun-Passives" deviceset="CAP_POL" device="PTH2"/>
 <part name="R1" library="SparkFun-Passives" deviceset="RESISTOR" device="PTH-1/4W" value="10k"/>
@@
 <part name="SJ2" library="jumper" deviceset="SJ" device=""/>
 <part name="U3" library="adafruit" deviceset="PINHD-1X10" device="" value="XBee Connector"/>
+<part name="JP6" library="screwterms" deviceset="SCREWTERM-2" device="" value="5V OUT"/>
 </parts>
 <sheets>
 <sheet>
 <plain>
-<text x="7.62" y="177.8" size="1.778" layer="97">J-Type Range = -180°C to 750°C</text>
-<text x="7.62" y="175.26" size="1.778" layer="97">K-Type Range = -180°C to 1200°C</text>
-<text x="7.62" y="170.18" size="1.778" layer="97">With a Single 5V Supply:</text>
-<text x="7.62" y="160.02" size="1.778" layer="97">1.24V REF = -248°C to 752°C</text>
-<text x="7.62" y="162.56" size="1.778" layer="97">0.9V REF = -180°C to 820°C</text>
-<text x="7.62" y="165.1" size="1.778" layer="97">0V REF = 0°C to 1000°C</text>
 </plain>
 <instances>
@@
 <instance part="U$8" gate="G$1" x="0" y="0"/>
 <instance part="U$9" gate="G$1" x="191.77" y="24.13"/>
-<instance part="JP1" gate="G$1" x="99.06" y="43.18" rot="R180"/>
+<instance part="JP1" gate="G$1" x="99.06" y="43.18"/>
 <instance part="U1" gate="G$1" x="73.66" y="129.54" smashed="yes"/>
 <instance part="U2" gate="G$1" x="185.42" y="129.54"/>
-<instance part="JP2" gate="G$1" x="124.46" y="43.18" rot="R180"/>
-<instance part="JP3" gate="G$1" x="99.06" y="20.32" rot="R180"/>
-<instance part="JP4" gate="G$1" x="124.46" y="20.32" rot="R180"/>
-<instance part="JP5" gate="G$1" x="121.92" y="58.42"/>
+<instance part="JP2" gate="G$1" x="124.46" y="43.18"/>
+<instance part="JP3" gate="G$1" x="99.06" y="20.32"/>
+<instance part="JP4" gate="G$1" x="124.46" y="20.32"/>
+<instance part="JP5" gate="G$1" x="132.08" y="58.42" rot="MR0"/>
 <instance part="C1" gate="G$1" x="101.6" y="60.96"/>
 <instance part="R1" gate="G$1" x="35.56" y="121.92"/>
@@
 <instance part="SJ2" gate="1" x="142.24" y="111.76"/>
 <instance part="U3" gate="G$1" x="162.56" y="78.74"/>
+<instance part="JP6" gate="G$1" x="93.98" y="81.28"/>
 </instances>
 <busses>
@@
 </segment>
 <segment>
-<pinref part="JP5" gate="G$1" pin="2"/>
-<wire x1="116.84" y1="58.42" x2="109.22" y2="58.42" width="0.1524" layer="91"/>
-<label x="111.76" y="58.42" size="1.778" layer="95"/>
+<pinref part="JP5" gate="G$1" pin="1"/>
+<wire x1="124.46" y1="55.88" x2="109.22" y2="55.88" width="0.1524" layer="91"/>
+<label x="116.84" y="55.88" size="1.778" layer="95" rot="MR0"/>
 <pinref part="C1" gate="G$1" pin="-"/>
 <wire x1="101.6" y1="55.88" x2="101.6" y2="53.34" width="0.1524" layer="91"/>
 <wire x1="101.6" y1="53.34" x2="109.22" y2="53.34" width="0.1524" layer="91"/>
-<wire x1="109.22" y1="53.34" x2="109.22" y2="58.42" width="0.1524" layer="91"/>
+<wire x1="109.22" y1="53.34" x2="109.22" y2="55.88" width="0.1524" layer="91"/>
 </segment>
 <segment>
@@
 <label x="147.32" y="81.28" size="1.778" layer="95"/>
 </segment>
+<segment>
+<pinref part="JP6" gate="G$1" pin="1"/>
+<wire x1="101.6" y1="78.74" x2="109.22" y2="78.74" width="0.1524" layer="91"/>
+<label x="106.68" y="78.74" size="1.778" layer="95"/>
+</segment>
 </net>
 <net name="2-B2" class="0">
@@
 </segment>
 <segment>
-<pinref part="JP4" gate="G$1" pin="2"/>
-<wire x1="129.54" y1="20.32" x2="137.16" y2="20.32" width="0.1524" layer="91"/>
-<label x="134.62" y="20.32" size="1.778" layer="95"/>
+<pinref part="JP4" gate="G$1" pin="1"/>
+<wire x1="132.08" y1="17.78" x2="137.16" y2="17.78" width="0.1524" layer="91"/>
+<label x="134.62" y="17.78" size="1.778" layer="95"/>
 </segment>
 </net>
@@
 </segment>
 <segment>
-<pinref part="JP4" gate="G$1" pin="1"/>
-<wire x1="129.54" y1="17.78" x2="137.16" y2="17.78" width="0.1524" layer="91"/>
-<label x="134.62" y="17.78" size="1.778" layer="95"/>
+<pinref part="JP4" gate="G$1" pin="2"/>
+<wire x1="132.08" y1="22.86" x2="137.16" y2="22.86" width="0.1524" layer="91"/>
+<label x="134.62" y="22.86" size="1.778" layer="95"/>
 </segment>
 </net>
@@
 </segment>
 <segment>
-<pinref part="JP3" gate="G$1" pin="1"/>
-<wire x1="104.14" y1="17.78" x2="111.76" y2="17.78" width="0.1524" layer="91"/>
-<label x="109.22" y="17.78" size="1.778" layer="95"/>
+<pinref part="JP3" gate="G$1" pin="2"/>
+<wire x1="106.68" y1="22.86" x2="111.76" y2="22.86" width="0.1524" layer="91"/>
+<label x="109.22" y="22.86" size="1.778" layer="95"/>
 </segment>
 </net>
@@
 </segment>
 <segment>
-<pinref part="JP3" gate="G$1" pin="2"/>
-<wire x1="104.14" y1="20.32" x2="111.76" y2="20.32" width="0.1524" layer="91"/>
-<label x="109.22" y="20.32" size="1.778" layer="95"/>
+<pinref part="JP3" gate="G$1" pin="1"/>
+<wire x1="106.68" y1="17.78" x2="111.76" y2="17.78" width="0.1524" layer="91"/>
+<label x="109.22" y="17.78" size="1.778" layer="95"/>
 </segment>
 </net>
@@
 <label x="147.32" y="76.2" size="1.778" layer="95"/>
 </segment>
+<segment>
+<pinref part="U2" gate="G$1" pin="RES"/>
+<wire x1="170.18" y1="127" x2="162.56" y2="127" width="0.1524" layer="91"/>
+<label x="160.02" y="127" size="1.778" layer="95"/>
+</segment>
+<segment>
+<pinref part="U1" gate="G$1" pin="RES"/>
+<wire x1="58.42" y1="127" x2="50.8" y2="127" width="0.1524" layer="91"/>
+<label x="48.26" y="127" size="1.778" layer="95"/>
+</segment>
+<segment>
+<pinref part="JP6" gate="G$1" pin="2"/>
+<wire x1="101.6" y1="83.82" x2="109.22" y2="83.82" width="0.1524" layer="91"/>
+<label x="106.68" y="83.82" size="1.778" layer="95"/>
+</segment>
 </net>
 <net name="2-MS1" class="0">
@@
 <wire x1="78.74" y1="53.34" x2="86.36" y2="53.34" width="0.1524" layer="91"/>
 <label x="81.28" y="53.34" size="1.778" layer="95"/>
-</segment>
-</net>
-<net name="2-RES" class="0">
-<segment>
-<pinref part="U2" gate="G$1" pin="RES"/>
-<wire x1="170.18" y1="127" x2="162.56" y2="127" width="0.1524" layer="91"/>
-<label x="160.02" y="127" size="1.778" layer="95"/>
 </segment>
 </net>
@@
 </segment>
 <segment>
-<pinref part="JP1" gate="G$1" pin="2"/>
-<wire x1="104.14" y1="43.18" x2="111.76" y2="43.18" width="0.1524" layer="91"/>
-<label x="109.22" y="43.18" size="1.778" layer="95"/>
+<pinref part="JP1" gate="G$1" pin="1"/>
+<wire x1="106.68" y1="40.64" x2="111.76" y2="40.64" width="0.1524" layer="91"/>
+<label x="109.22" y="40.64" size="1.778" layer="95"/>
 </segment>
 </net>
@@
 </segment>
 <segment>
-<pinref part="JP1" gate="G$1" pin="1"/>
-<wire x1="104.14" y1="40.64" x2="111.76" y2="40.64" width="0.1524" layer="91"/>
-<label x="109.22" y="40.64" size="1.778" layer="95"/>
+<pinref part="JP1" gate="G$1" pin="2"/>
+<wire x1="106.68" y1="45.72" x2="111.76" y2="45.72" width="0.1524" layer="91"/>
+<label x="109.22" y="45.72" size="1.778" layer="95"/>
 </segment>
 </net>
@@
 </segment>
 <segment>
-<pinref part="JP2" gate="G$1" pin="1"/>
-<wire x1="129.54" y1="40.64" x2="137.16" y2="40.64" width="0.1524" layer="91"/>
-<label x="134.62" y="40.64" size="1.778" layer="95"/>
+<pinref part="JP2" gate="G$1" pin="2"/>
+<wire x1="132.08" y1="45.72" x2="137.16" y2="45.72" width="0.1524" layer="91"/>
+<label x="134.62" y="45.72" size="1.778" layer="95"/>
 </segment>
 </net>
@@
 </segment>
 <segment>
-<pinref part="JP2" gate="G$1" pin="2"/>
-<wire x1="129.54" y1="43.18" x2="137.16" y2="43.18" width="0.1524" layer="91"/>
-<label x="134.62" y="43.18" size="1.778" layer="95"/>
+<pinref part="JP2" gate="G$1" pin="1"/>
+<wire x1="132.08" y1="40.64" x2="137.16" y2="40.64" width="0.1524" layer="91"/>
+<label x="134.62" y="40.64" size="1.778" layer="95"/>
 </segment>
 </net>
@@
 <wire x1="78.74" y1="27.94" x2="86.36" y2="27.94" width="0.1524" layer="91"/>
 <label x="81.28" y="27.94" size="1.778" layer="95"/>
-</segment>
-</net>
-<net name="1-RES" class="0">
-<segment>
-<pinref part="U1" gate="G$1" pin="RES"/>
-<wire x1="58.42" y1="127" x2="50.8" y2="127" width="0.1524" layer="91"/>
-<label x="48.26" y="127" size="1.778" layer="95"/>
 </segment>
 </net>
@@
 <net name="+12V" class="0">
 <segment>
-<pinref part="JP5" gate="G$1" pin="1"/>
-<wire x1="116.84" y1="60.96" x2="109.22" y2="60.96" width="0.1524" layer="91"/>
+<pinref part="JP5" gate="G$1" pin="2"/>
+<wire x1="124.46" y1="60.96" x2="109.22" y2="60.96" width="0.1524" layer="91"/>
 <label x="111.76" y="60.96" size="1.778" layer="95"/>
 <wire x1="109.22" y1="60.96" x2="109.22" y2="66.04" width="0.1524" layer="91"/>
